Commit message: No imu mode, hokuyo roll flip!

File: orne_description/urdf/orne_alpha.xacro (robot description, xacro)
@@ -14,5 +14,5 @@
 <!-- Setting for levelly fixed 2D URG -->
 <xacro:sensor_hokuyo name="hokuyo" parent="base_link">
-    <origin xyz="0.212 0 0.2485" rpy="0 0 0"/>
+    <origin xyz="0.212 0 0.2485" rpy="3.14 0 0"/>
 </xacro:sensor_hokuyo>
 <!-- Setting for diagonally fixed 2D URG -->
