Commit message: Changes made to xacro for icart mini

File: orne_description/urdf/orne_v.xacro (robot description, xacro)
@@ -5,10 +5,10 @@
                          xmlns:interface="http://playerstage.sourceforge.net/gazebo/xmlschema/#interface"
 >
-<xacro:include filename="$(find orne_description)/urdf/orne_x.xacro"/>
+<xacro:include filename="$(find icart_mini_description)/urdf/icart_mini.xacro"/>
 <xacro:include filename="$(find icart_mini_description)/urdf/sensors/imu.urdf.xacro"/>
 <xacro:include filename="$(find icart_mini_description)/urdf/sensors/hokuyo.urdf.xacro"/>
 <!-- Setting for imu -->
 <xacro:sensor_imu name="imu" parent="base_link" size="0.05 0.05 0.05">
-    <origin xyz="-0.145 0.0 0.21" rpy="0 0 0"/>
+    <origin xyz="-0.0 0.0 0.1" rpy="0 0 0"/>
 </xacro:sensor_imu>
 <!-- Setting for levelly fixed 2D URG -->
@@ -16,14 +16,3 @@
     <origin xyz="0.212 0 0.2485" rpy="0 0 0"/>
 </xacro:sensor_hokuyo>
-<!-- Setting for diagonally fixed 2D URG -->
-<xacro:include filename="$(find icart_mini_description)/urdf/sensors/hokuyo.urdf.xacro"/>
-<xacro:sensor_hokuyo name="diagonally_hokuyo" parent="base_link">
-   <origin xyz="0.098 0 0.422" rpy="0 0.296706 0"/>
-</xacro:sensor_hokuyo>
-<!--
-<xacro:include filename="$(find icart_mini_description)/urdf/sensors/hokuyo3d.urdf.xacro"/>
-<xacro:sensor_hokuyo3d name="hokuyo3d" parent="base_link">
-    <origin xyz="0.12 0 0.35" rpy="0 0.192 0"/>
-</xacro:sensor_hokuyo3d>
--->
 </robot>

Commit message: Got the imugit add --all!

File: orne_description/urdf/orne_v.xacro (robot description, xacro)
@@ -10,5 +10,5 @@
 <!-- Setting for imu -->
 <xacro:sensor_imu name="imu" parent="base_link" size="0.05 0.05 0.05">
-    <origin xyz="-0.0 0.0 0.1" rpy="0 0 0"/>
+    <origin xyz="-0.0 0.0 0.1" rpy="0 3.14 0"/>
 </xacro:sensor_imu>
 <!-- Setting for levelly fixed 2D URG -->
